File: BatAger.sch (KiCad schematic (older format))
At the start: 22 parts

Commit message: modified:   BatAger-cache.lib 	modified:   BatAger.pro 	modified:   BatAger.sch 	new file:   lib/Gajda_amplif.lib
Parts:
- added U?: LM358DUAL, symbol LM358DUAL
Connections:
- wire segments 29 -> 27
Other:
- moved on the sheet: Q?, R?
Changed lines of the file:
@@
 LIBS:contrib
 LIBS:valves
+LIBS:Gajda_amplif
 LIBS:BatAger-cache
 EELAYER 27 0
@@
 L BTS141 Q?
 U 1 1 561B703D
-P 8700 2750
-F 0 "Q?" H 8900 2825 50  0000 L CNN
-F 1 "CSD18536KCS" H 8900 2750 50  0000 L CNN
-F 2 "TO-220" H 8900 2675 50  0000 L CIN
-F 3 "" H 8700 2750 50  0000 L CNN
-	1    8700 2750
+P 8700 2900
+F 0 "Q?" H 8900 2975 50  0000 L CNN
+F 1 "CSD18536KCS" H 8900 2900 50  0000 L CNN
+F 2 "TO-220" H 8900 2825 50  0000 L CIN
+F 3 "" H 8700 2900 50  0000 L CNN
+	1    8700 2900
 	1    0    0    -1
 $EndComp
@@
 L R R?
 U 1 1 561B7F04
-P 9550 1600
-F 0 "R?" V 9630 1600 50  0000 C CNN
-F 1 "R" V 9550 1600 50  0000 C CNN
-F 2 "" V 9480 1600 30  0000 C CNN
-F 3 "" H 9550 1600 30  0000 C CNN
-	1    9550 1600
+P 9450 1600
+F 0 "R?" V 9530 1600 50  0000 C CNN
+F 1 "R" V 9450 1600 50  0000 C CNN
+F 2 "" V 9380 1600 30  0000 C CNN
+F 3 "" H 9450 1600 30  0000 C CNN
+	1    9450 1600
 	0    1    1    0
 $EndComp
@@
 L R R?
 U 1 1 561B8496
-P 9250 2350
-F 0 "R?" V 9330 2350 50  0000 C CNN
-F 1 "R" V 9250 2350 50  0000 C CNN
-F 2 "" V 9180 2350 30  0000 C CNN
-F 3 "" H 9250 2350 30  0000 C CNN
-	1    9250 2350
+P 9250 2500
+F 0 "R?" V 9330 2500 50  0000 C CNN
+F 1 "R" V 9250 2500 50  0000 C CNN
+F 2 "" V 9180 2500 30  0000 C CNN
+F 3 "" H 9250 2500 30  0000 C CNN
+	1    9250 2500
 	0    1    1    0
 $EndComp
@@
 L GND #PWR?
 U 1 1 561B8F91
-P 8800 2950
-F 0 "#PWR?" H 8800 2700 50  0001 C CNN
-F 1 "GND" H 8800 2800 50  0000 C CNN
-F 2 "" H 8800 2950 60  0000 C CNN
-F 3 "" H 8800 2950 60  0000 C CNN
-	1    8800 2950
+P 8800 3100
+F 0 "#PWR?" H 8800 2850 50  0001 C CNN
+F 1 "GND" H 8800 2950 50  0000 C CNN
+F 2 "" H 8800 3100 60  0000 C CNN
+F 3 "" H 8800 3100 60  0000 C CNN
+	1    8800 3100
 	1    0    0    -1
 $EndComp
@@
 L R R?
 U 1 1 561B905E
-P 8350 2800
-F 0 "R?" V 8430 2800 50  0000 C CNN
-F 1 "R" V 8350 2800 50  0000 C CNN
-F 2 "" V 8280 2800 30  0000 C CNN
-F 3 "" H 8350 2800 30  0000 C CNN
-	1    8350 2800
+P 8350 2950
+F 0 "R?" V 8430 2950 50  0000 C CNN
+F 1 "R" V 8350 2950 50  0000 C CNN
+F 2 "" V 8280 2950 30  0000 C CNN
+F 3 "" H 8350 2950 30  0000 C CNN
+	1    8350 2950
 	0    1    1    0
 $EndComp
@@
 	8900 1700 9900 1700
 Wire Wire Line
-	9100 2000 9100 2350
-Wire Wire Line
-	9400 1600 9400 2350
-Wire Wire Line
-	11200 1150 10550 1150
-Wire Wire Line
 	11200 1700 11200 1150
 Wire Wire Line
@@
 	9700 1150 9700 1600
 Wire Wire Line
-	10250 1150 9700 1150
-Wire Wire Line
-	8800 2350 8800 2550
-Wire Wire Line
-	9100 2350 8800 2350
+	8800 2500 8800 2700
 Wire Wire Line
 	7650 1450 7650 1550
@@
 Wire Wire Line
 	8900 4450 8950 4450
+Wire Wire Line
+	11200 1150 10650 1150
+Wire Wire Line
+	10150 1150 9700 1150
+Wire Wire Line
+	8800 2500 9000 2500
+$Comp
+L LM358DUAL U?
+U 1 1 561BA7F0
+P 5800 4950
+F 0 "U?" H 5950 5200 60  0000 L CNN
+F 1 "LM358DUAL" H 5800 4450 60  0000 L CNN
+F 2 "" H 5800 4950 60  0000 C CNN
+F 3 "" H 5800 4950 60  0000 C CNN
+	1    5800 4950
+	1    0    0    -1
+$EndComp
 $EndSCHEMATC
