File: pcb/BatAger.kicad_pcb (KiCad board)
At the start: 2 copper layers, 159 parts, among them CON1 AVR-ISP-6, IC1 ATMEGA2560-A, P1 FTDI, P10 CONN_01X02, P11 CONN_01X02, P12 CONN_01X02, P13 -15V, P14 GND, P15 AUX, P2 +15V, P3 BAT1_TP, P4 BAT3_TP, P5 BAT5_TP, P6 BAT2_TP, P7 BAT4_TP, P8 CONN_01X02, P9 CONN_01X02, Q1 IRFR3607PBF, Q10 BC849, Q11 IRF9530, Q12 BC849, Q13 CSD18536KCS, Q14 BC849, Q15 IRF9530, Q16 BC849, Q17 CSD18536KCS, Q18 BC849, Q19 IRF9530, Q2 BC849, Q20 BC849, Q21 CSD18536KCS, Q3 IRF9530, Q4 CSD18536KCS, Q5 BC849, Q6 BC849, Q7 IRF9530, Q8 CSD18536KCS, Q9 BC849, SW1 SW_PUSH_4PIN, U1 MC33269, U2 LM358DUAL, U3 LM358DUAL, U4 LM358DUAL, U5 LM358DUAL, U6 LM358DUAL, Y1 16MHz

Commit message: last commit before starting traces
Parts:
- R61: footprint Resistors_SMD:R_2512_HandSoldering -> Resistors_SMD:R_0805_HandSoldering
- moved R74 136.9 mm to (260.4, 26.0), turned to 90 degrees
- moved R68 133.8 mm to (256.5, 26.0), turned to 90 degrees
- moved P12 133.5 mm to (249.6, 17.8), turned to 90 degrees
- moved R67 129.0 mm to (260.4, 40.6), turned to 90 degrees
- moved R79 127.1 mm to (249.6, 27.9), turned to 270 degrees
- moved R71 126.3 mm to (257.2, 40.6), turned to 270 degrees
- moved P5 125.2 mm to (270.5, 76.8)
- moved Q19 120.5 mm to (249.6, 39.4), turned to 180 degrees
- moved R80 120.2 mm to (241.3, 28.6), turned to 270 degrees
- moved U6 119.5 mm to (257.2, 55.2)
- moved C21 119.4 mm to (259.7, 61.6), turned to 180 degrees
- moved R70 116.3 mm to (260.4, 73.0), turned to 270 degrees
- moved C22 114.1 mm to (254.0, 61.6)
- moved R69 112.7 mm to (256.5, 73.0), turned to 90 degrees
- moved R76 112.4 mm to (245.1, 47.6), turned to 270 degrees
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Connections:
- R79 pad 1: (no net) -> /Sheet561DD110/bat5+
- R79 pad 2: (no net) -> /Sheet561DD110/shunt5_high

Commit message: trace complete (maybe!)
Parts:
- moved P3 47.9 mm to (100.1, 53.3), turned to 180 degrees
- moved P4 34.4 mm to (199.1, 55.4), turned to 180 degrees
- moved P6 29.5 mm to (148.8, 55.4), turned to 180 degrees
- moved C21 28.6 mm to (286.9, 70.4)
- moved C22 28.6 mm to (281.2, 70.4)
- moved R69 28.6 mm to (283.7, 81.8)
- moved R70 28.6 mm to (287.5, 81.8)
- moved U6 28.6 mm to (284.4, 64.0)
- moved Q21 27.1 mm to (274.7, 94.9)
- moved R18 26.7 mm to (70.0, 77.5), turned to 90 degrees
- moved P12 26.6 mm to (274.6, 26.7)
- moved Q19 26.6 mm to (274.6, 48.3), turned to 0 degrees
- moved R67 26.6 mm to (285.4, 49.5)
- moved R68 26.6 mm to (281.6, 34.9)
- moved R71 26.6 mm to (282.2, 49.5)
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Connections:
- CON1 pad 5: (no net) -> /RESET
- IC1 pad 1: /CC2 -> /Sheet561CB83A/chg_ctrl2
- P6 pad 1: /CC2 -> /Sheet561CB83A/chg_ctrl2
- R27 pad 1: /Sheet561CB83A/chg_ctrl1 -> /Sheet561CB83A/chg_ctrl2
- R28 pad 2: /Sheet561CB83A/chg_ctrl1 -> /Sheet561CB83A/chg_ctrl2
- U3 pad 1: (no net) -> Net-(R29-Pad2)
- U3 pad 2: (no net) -> Net-(R23-Pad1)
- U3 pad 3: (no net) -> Net-(R22-Pad1)
- U3 pad 5: Net-(R22-Pad1) -> Net-(R29-Pad2)
- U3 pad 7: Net-(R29-Pad2) -> /Sheet561CB83A/i2
- U5 pad 1: (no net) -> Net-(R59-Pad2)
- U5 pad 2: (no net) -> Net-(R53-Pad1)
- U5 pad 3: (no net) -> Net-(R52-Pad1)
- U5 pad 5: Net-(R52-Pad1) -> Net-(R59-Pad2)
- U5 pad 6: Net-(R53-Pad1) -> Net-(R54-Pad2)
- U5 pad 7: Net-(R59-Pad2) -> /Sheet561D4A90/i4
Routing:
- net VCC: track 0.00 -> 428.3 mm, vias 0 -> 11
- net -15V: track 0.00 -> 343.8 mm, vias 0 -> 7
- net /Sheet561DD110/dchg_ctrl5: track 0.00 -> 281.8 mm, vias 0 -> 3
- net /Sheet561DD110/vbat5: track 0.00 -> 278.4 mm, vias 0 -> 1
- net /Sheet561DD110/chg_ctrl5: track 0.00 -> 275.1 mm, vias 0 -> 5
- net /Sheet561DD110/dc_led5: track 0.00 -> 271.5 mm, vias 0 -> 3
- net /Sheet561DD110/i5: track 0.00 -> 257.7 mm, vias 0 -> 2
- net /Sheet561D4A90/dchg_ctrl4: track 0.00 -> 252.9 mm, vias 0 -> 4
- net /Sheet561D4A90/vbat4: track 0.00 -> 245.6 mm, vias 0 -> 2
- net /Sheet561D4A90/chg_ctrl4: track 0.00 -> 220.0 mm, vias 0 -> 6
- net /Sheet561D4A90/dc_led4: track 0.00 -> 217.8 mm, vias 0 -> 2
- net /Sheet561D4A90/dchg_ctrl3: track 0.00 -> 213.5 mm, vias 0 -> 3
- net /Sheet561D4A90/i4: track 0.00 -> 211.4 mm, vias 0 -> 2
- net /Sheet561D4A90/dc_led3: track 0.00 -> 203.7 mm, vias 0 -> 5
- net /Sheet561D4A90/chg_ctrl3: track 0.00 -> 192.2 mm, vias 0 -> 6
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- added copper zone on F.Cu, net GND
Other:
- net class Default: clearance 0.3048 -> 0.1524
- net class Default2 added: clearance 0.3048, trace_width 0.3048, via_dia 0.508, via_drill 0.4064
- net class High_current: trace_width 0.762 -> 2.032
- net class Power: clearance 0.3048 -> 0.127
- rule trace_clearance: 0.3048 -> 0.1524

Commit message: done for today. i1 & i2 still unconnected.
Parts:
- moved R15 0.99 mm to (73.2, 55.1), turned to 270 degrees
- turned Q3 to 0 degrees
- turned Q7 to 0 degrees
Routing:
- net +15V: track 68.3 -> 252.5 mm, vias 0 -> 20
- net Net-(Q2-Pad3): track 0.00 -> 15.7 mm
- net Net-(Q6-Pad3): track 9.45 -> 19.5 mm
- added copper zone on B.Cu, net +15V

Commit message: adding planes - almost done!
Parts:
- added P16: FAN, Pin_Headers:Pin_Header_Straight_1x02, F.Cu at (103.6, 94.7)
- added Q22: CSD18536KCS, Power_Integrations:TO-220, F.Cu at (105.9, 77.5)
- added R82: 220, Resistors_SMD:R_0805_HandSoldering, F.Cu at (98.8, 77.0)
- moved C15 12.3 mm to (144.5, 57.1), turned to 90 degrees
- moved C17 11.0 mm to (192.8, 59.9)
- moved C10 1.40 mm to (46.0, 57.4), turned to 0 degrees
Connections:
- IC1 pad 42: (no net) -> /Sheet561DD110/fan_ctrl
Routing:
- net GND: track 3.22 -> 163.6 mm, vias 0 -> 4
- net /Sheet561CB83A/i2: track 23.2 -> 137.8 mm, vias 0 -> 2
- net /Sheet561CB83A/i1: track 26.4 -> 91.4 mm, vias 0 -> 2
- net /Sheet561DD110/fan_ctrl: track 0.00 -> 64.5 mm, vias 0 -> 4
- net Net-(P16-Pad2): track 0.00 -> 17.4 mm
- net Net-(R69-Pad2): track 3.81 -> 19.6 mm
- net VCC: track 428.3 -> 442.1 mm, vias 11 -> 13
- net /Sheet561CB83A/vbat2: track 133.2 -> 143.0 mm, vias 1 -> 2
- net +15V: track 252.5 -> 243.9 mm, vias 20 -> 17
- net Net-(Q22-Pad1): track 0.00 -> 4.92 mm
- net /Sheet561CB83A/chg_ctrl2: track 137.3 -> 141.9 mm
- net /Sheet561D4A90/i3: track 182.6 -> 183.4 mm
- net /Sheet561D4A90/i4: track 211.4 -> 212.2 mm
Other:
- net class Default: clearance 0.1524 -> 0.0254
- net class Default2 removed
- rule trace_clearance: 0.1524 -> 0.0254

Commit message: going to change drill sizes.
Routing:
- net GND: track 163.6 -> 203.9 mm, vias 4 -> 10
Other:
- board outline added: 285.8 x 74.9 mm

Commit message: Production candidate - passes DRC.
Parts:
- added REF**: 1pin, Connect:1pin, F.Cu at (17.8, 29.2)
- added REF**: 1pin, Connect:1pin, F.Cu at (16.5, 92.7)
- added REF**: 1pin, Connect:1pin, F.Cu at (292.1, 92.7)
- added REF**: 1pin, Connect:1pin, F.Cu at (292.1, 26.7)
- added REF**: 1pin, Connect:1pin, F.Cu at (152.4, 94.0)
- added REF**: 1pin, Connect:1pin, F.Cu at (152.4, 27.9)
- C11, C12: footprint Capacitors_Elko_ThroughHole:Elko_vert_11.5x8mm_RM3.5 -> Custom Footprints:Elko_vert_11.5x8mm_RM3.5
- R10, R11, R14, R20, R21, R22, R23, R24, R25, R26, R29, R35, R36, R37, R38, R39, R40, R41, R50, R51, R52, R53, R54, R55, R56, R59, R65, R66, R67, R68, R69, R7, R70, R71, R74, R8, R80, R81, R9: footprint Resistors_ThroughHole:Resistor_Horizontal_RM10mm -> Custom Footprints:Resistor_Horizontal_RM10mm

Commit message: Reduced number of drill sizes.
Parts:
- Q11, Q13, Q15, Q17, Q19, Q21, Q22, Q3, Q4, Q7, Q8: footprint Power_Integrations:TO-220 -> Custom Footprints:TO-220
Routing:
- net (no net): track 1.57 -> 0.00 mm
- net GND: track 203.9 -> 204.7 mm

Commit message: Changed fan FET (Q22). Many other minor layout changes. Production candidate.
Parts:
- added Q23: BC849, Housings_SOT-23_SOT-143_TSOT-6:SOT-23_Handsoldering, F.Cu at (97.7, 72.4)
- added Q24: BC849, Housings_SOT-23_SOT-143_TSOT-6:SOT-23_Handsoldering, F.Cu at (107.7, 75.6)
- added R83: 200, Resistors_SMD:R_0805_HandSoldering, F.Cu at (112.4, 76.1)
- added R84: 1k, Resistors_SMD:R_0805_HandSoldering, F.Cu at (103.4, 77.1)
- Q22: value CSD18536KCS -> IRFR3607PBF; footprint Custom Footprints:TO-220 -> TO_SOT_Packages_SMD:TO-252-2Lead
- R12, R27, R32, R33, R42, R47, R48, R57, R62, R63, R72, R77, R78: value R -> 200
- R13, R16: value 200 -> 1k
- R15, R28, R30, R31, R43, R45, R46, R58, R60, R61, R73, R75, R76: value R -> 1k
- R19, R34: value R -> 0R056
- R44: footprint Resistors_ThroughHole:Resistor_Horizontal_RM10mm -> Custom Footprints:Resistor_Horizontal_RM10mm
- R82: value 220 -> 200
- SW1: footprint Buttons_Switches_ThroughHole:SW_PUSH_SMALL -> Custom Footprints:SW_PUSH_4.5x6.5mm
- Y1: footprint Crystals:Crystal_HC48-U_Vertical -> Crystals:Crystal_HC49-U_Vertical
- moved R62 17.5 mm to (233.4, 93.6), turned to 90 degrees
- moved R47 16.7 mm to (184.9, 92.1)
- moved R32 14.2 mm to (134.2, 91.1)
- moved R77 12.2 mm to (279.7, 87.1), turned to 90 degrees
- moved R17 11.5 mm to (85.3, 90.6)
- moved Q22 3.58 mm to (106.9, 80.9), turned to 180 degrees
- moved SW1 2.42 mm to (23.7, 82.4)
- moved R82 2.41 mm to (96.5, 77.7), turned to 270 degrees
- moved Y1 2.41 mm to (36.8, 92.7)
- moved REF** 1.80 mm to (16.5, 27.9)
- moved REF** 1.27 mm to (292.1, 27.9)
- turned Q13 to 180 degrees
- turned Q17 to 180 degrees
- turned Q21 to 180 degrees
- turned Q4 to 180 degrees
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Connections:
- R82 pad 1: Net-(Q22-Pad1) -> Net-(Q23-Pad1)
- U2 pad 5: Net-(R14-Pad2) -> Net-(R10-Pad1)
- U2 pad 6: Net-(R10-Pad1) -> Net-(R14-Pad2)
- U3 pad 5: Net-(R29-Pad2) -> Net-(R24-Pad2)
- U3 pad 6: Net-(R24-Pad2) -> Net-(R29-Pad2)
- U4 pad 5: Net-(R44-Pad2) -> Net-(R39-Pad2)
- U4 pad 6: Net-(R39-Pad2) -> Net-(R44-Pad2)
- U5 pad 5: Net-(R59-Pad2) -> Net-(R54-Pad2)
- U5 pad 6: Net-(R54-Pad2) -> Net-(R59-Pad2)
- U6 pad 5: Net-(R74-Pad2) -> Net-(R69-Pad2)
- U6 pad 6: Net-(R69-Pad2) -> Net-(R74-Pad2)
Routing:
- net GND: track 204.7 -> 277.7 mm, vias 10 -> 13
- net Net-(Q23-Pad3): track 0.00 -> 20.3 mm, vias 0 -> 2
- net /Sheet561D4A90/dchg_ctrl3: track 213.5 -> 232.3 mm, vias 3 -> 4
- net /Sheet561CB83A/dchg_ctrl2: track 160.3 -> 176.1 mm, vias 5 -> 7
- net /Sheet561CB83A/dchg_ctrl1: track 121.5 -> 134.9 mm, vias 4 -> 6
- net Net-(P16-Pad2): track 17.4 -> 7.81 mm
- net +15V: track 243.9 -> 237.1 mm
- net VCC: track 442.1 -> 437.9 mm, vias 13 -> 14
- net /Sheet561DD110/dchg_ctrl5: track 281.8 -> 285.7 mm
- net /Sheet561D4A90/dchg_ctrl4: track 252.9 -> 256.4 mm, vias 4 -> 2
- net /Sheet561DD110/fan_ctrl: track 64.5 -> 61.1 mm
- net Net-(R74-Pad2): track 50.2 -> 46.8 mm
- net Net-(Q23-Pad1): track 0.00 -> 2.56 mm
- net Net-(Q22-Pad1): track 4.92 -> 7.44 mm
- net Net-(R24-Pad2): track 25.8 -> 23.7 mm
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