File: pcb/file561D4A90.sch (KiCad schematic (older format))
At the start: 52 parts, among them P10 CONN_01X02, P11 CONN_01X02, Q10 BC849, Q11 IRF9530, Q12 BC849, Q13 CSD18536KCS, Q14 BC849, Q15 IRF9530, Q16 BC849, Q17 CSD18536KCS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

Commit message: Changed R62 & C26 to PTH.
Parts:
- C26: footprint Capacitors_SMD:C_0805_HandSoldering -> Capacitors_ThroughHole:C_Disc_D3_P2.5
- R62: footprint Resistors_SMD:R_0805_HandSoldering -> Custom Footprints:Resistor_Horizontal_RM10mm
Changed lines of the file:
@@
 $EndComp
 $Comp
-L +15V #PWR75
+L +15V #PWR055
 U 1 1 561D540A
 P 3700 800
-F 0 "#PWR75" H 3700 650 50  0001 C CNN
+F 0 "#PWR055" H 3700 650 50  0001 C CNN
 F 1 "+15V" H 3700 940 50  0000 C CNN
 F 2 "" H 3700 800 60  0000 C CNN
@@
 $EndComp
 $Comp
-L GND-RESCUE-BatAger #PWR71
+L GND-RESCUE-BatAger #PWR056
 U 1 1 561D5410
 P 3050 1450
-F 0 "#PWR71" H 3050 1200 50  0001 C CNN
+F 0 "#PWR056" H 3050 1200 50  0001 C CNN
 F 1 "GND" H 3050 1300 50  0000 C CNN
 F 2 "" H 3050 1450 60  0000 C CNN
@@
 $EndComp
 $Comp
-L GND-RESCUE-BatAger #PWR79
+L GND-RESCUE-BatAger #PWR057
 U 1 1 561D541D
 P 4300 2600
-F 0 "#PWR79" H 4300 2350 50  0001 C CNN
+F 0 "#PWR057" H 4300 2350 50  0001 C CNN
 F 1 "GND" H 4300 2450 50  0000 C CNN
 F 2 "" H 4300 2600 60  0000 C CNN
@@
 $EndComp
 $Comp
-L GND-RESCUE-BatAger #PWR78
+L GND-RESCUE-BatAger #PWR058
 U 1 1 561D5431
 P 4200 4550
-F 0 "#PWR78" H 4200 4300 50  0001 C CNN
+F 0 "#PWR058" H 4200 4300 50  0001 C CNN
 F 1 "GND" H 4200 4400 50  0000 C CNN
 F 2 "" H 4200 4550 60  0000 C CNN
@@
 $EndComp
 $Comp
-L GND-RESCUE-BatAger #PWR68
+L GND-RESCUE-BatAger #PWR059
 U 1 1 561D5437
 P 2150 2300
-F 0 "#PWR68" H 2150 2050 50  0001 C CNN
+F 0 "#PWR059" H 2150 2050 50  0001 C CNN
 F 1 "GND" H 2150 2150 50  0000 C CNN
 F 2 "" H 2150 2300 60  0000 C CNN
@@
 $EndComp
 $Comp
-L +15V #PWR69
+L +15V #PWR060
 U 1 1 561D544B
 P 2400 2850
-F 0 "#PWR69" H 2400 2700 50  0001 C CNN
+F 0 "#PWR060" H 2400 2700 50  0001 C CNN
 F 1 "+15V" H 2400 2990 50  0000 C CNN
 F 2 "" H 2400 2850 60  0000 C CNN
@@
 $EndComp
 $Comp
-L GND-RESCUE-BatAger #PWR59
+L GND-RESCUE-BatAger #PWR061
 U 1 1 561D5465
 P 1100 4100
-F 0 "#PWR59" H 1100 3850 50  0001 C CNN
+F 0 "#PWR061" H 1100 3850 50  0001 C CNN
 F 1 "GND" H 1100 3950 50  0000 C CNN
 F 2 "" H 1100 4100 60  0000 C CNN
@@
 $EndComp
 $Comp
-L GND-RESCUE-BatAger #PWR63
+L GND-RESCUE-BatAger #PWR062
 U 1 1 561D5489
 P 1600 4900
-F 0 "#PWR63" H 1600 4650 50  0001 C CNN
+F 0 "#PWR062" H 1600 4650 50  0001 C CNN
 F 1 "GND" H 1600 4750 50  0000 C CNN
 F 2 "" H 1600 4900 60  0000 C CNN
@@
 $EndComp
 $Comp
-L VCC #PWR62
+L VCC #PWR063
 U 1 1 561D548F
 P 1600 3850
-F 0 "#PWR62" H 1600 3700 50  0001 C CNN
+F 0 "#PWR063" H 1600 3700 50  0001 C CNN
 F 1 "VCC" H 1600 4000 50  0000 C CNN
 F 2 "" H 1600 3850 60  0000 C CNN
@@
 	1900 1200 2250 1200
 $Comp
-L +15V #PWR74
+L +15V #PWR064
 U 1 1 561D54C5
 P 3350 1700
-F 0 "#PWR74" H 3350 1550 50  0001 C CNN
+F 0 "#PWR064" H 3350 1550 50  0001 C CNN
 F 1 "+15V" H 3350 1840 50  0000 C CNN
 F 2 "" H 3350 1700 60  0000 C CNN
@@
 	5100 3800 5100 3750
 $Comp
-L GND-RESCUE-BatAger #PWR80
+L GND-RESCUE-BatAger #PWR065
 U 1 1 561D54D3
 P 5100 4350
-F 0 "#PWR80" H 5100 4100 50  0001 C CNN
+F 0 "#PWR065" H 5100 4100 50  0001 C CNN
 F 1 "GND" H 5100 4200 50  0000 C CNN
 F 2 "" H 5100 4350 60  0000 C CNN
@@
 	3350 4250 3150 4250
 $Comp
-L VCC #PWR77
+L VCC #PWR066
 U 1 1 561D54E1
 P 4200 3050
-F 0 "#PWR77" H 4200 2900 50  0001 C CNN
+F 0 "#PWR066" H 4200 2900 50  0001 C CNN
 F 1 "VCC" H 4200 3200 50  0000 C CNN
 F 2 "" H 4200 3050 60  0000 C CNN
@@
 $EndComp
 $Comp
-L +15V #PWR91
+L +15V #PWR067
 U 1 1 561D8493
 P 9000 800
-F 0 "#PWR91" H 9000 650 50  0001 C CNN
+F 0 "#PWR067" H 9000 650 50  0001 C CNN
 F 1 "+15V" H 9000 940 50  0000 C CNN
 F 2 "" H 9000 800 60  0000 C CNN
@@
 $EndComp
 $Comp
-L GND-RESCUE-BatAger #PWR89
+L GND-RESCUE-BatAger #PWR068
 U 1 1 561D8499
 P 8350 1450
-F 0 "#PWR89" H 8350 1200 50  0001 C CNN
+F 0 "#PWR068" H 8350 1200 50  0001 C CNN
 F 1 "GND" H 8350 1300 50  0000 C CNN
 F 2 "" H 8350 1450 60  0000 C CNN
@@
 $EndComp
 $Comp
-L GND-RESCUE-BatAger #PWR95
+L GND-RESCUE-BatAger #PWR069
 U 1 1 561D84A5
 P 9600 2600
-F 0 "#PWR95" H 9600 2350 50  0001 C CNN
+F 0 "#PWR069" H 9600 2350 50  0001 C CNN
 F 1 "GND" H 9600 2450 50  0000 C CNN
 F 2 "" H 9600 2600 60  0000 C CNN
@@
 F 0 "R62" V 8980 2400 50  0000 C CNN
 F 1 "200" V 8900 2400 50  0000 C CNN
-F 2 "Resistors_SMD:R_0805_HandSoldering" V 8830 2400 30  0001 C CNN
+F 2 "Custom Footprints:Resistor_Horizontal_RM10mm" V 8830 2400 30  0001 C CNN
 F 3 "" H 8900 2400 30  0000 C CNN
 	1    8900 2400
@@
 $EndComp
 $Comp
-L GND-RESCUE-BatAger #PWR94
+L GND-RESCUE-BatAger #PWR070
 U 1 1 561D84B7
 P 9500 4550
-F 0 "#PWR94" H 9500 4300 50  0001 C CNN
+F 0 "#PWR070" H 9500 4300 50  0001 C CNN
 F 1 "GND" H 9500 4400 50  0000 C CNN
 F 2 "" H 9500 4550 60  0000 C CNN
@@
 $EndComp
 $Comp
-L GND-RESCUE-BatAger #PWR86
+L GND-RESCUE-BatAger #PWR071
 U 1 1 561D84BD
 P 7450 2300
-F 0 "#PWR86" H 7450 2050 50  0001 C CNN
+F 0 "#PWR071" H 7450 2050 50  0001 C CNN
 F 1 "GND" H 7450 2150 50  0000 C CNN
 F 2 "" H 7450 2300 60  0000 C CNN
@@
 $EndComp
 $Comp
-L +15V #PWR87
+L +15V #PWR072
 U 1 1 561D84CF
 P 7700 2750
-F 0 "#PWR87" H 7700 2600 50  0001 C CNN
+F 0 "#PWR072" H 7700 2600 50  0001 C CNN
 F 1 "+15V" H 7700 2890 50  0000 C CNN
 F 2 "" H 7700 2750 60  0000 C CNN
@@
 $EndComp
 $Comp
-L GND-RESCUE-BatAger #PWR81
+L GND-RESCUE-BatAger #PWR073
 U 1 1 561D84E7
 P 6400 4100
-F 0 "#PWR81" H 6400 3850 50  0001 C CNN
+F 0 "#PWR073" H 6400 3850 50  0001 C CNN
 F 1 "GND" H 6400 3950 50  0000 C CNN
 F 2 "" H 6400 4100 60  0000 C CNN
@@
 $EndComp
 $Comp
-L GND-RESCUE-BatAger #PWR83
+L GND-RESCUE-BatAger #PWR074
 U 1 1 561D8507
 P 6900 4900
-F 0 "#PWR83" H 6900 4650 50  0001 C CNN
+F 0 "#PWR074" H 6900 4650 50  0001 C CNN
 F 1 "GND" H 6900 4750 50  0000 C CNN
 F 2 "" H 6900 4900 60  0000 C CNN
@@
 $EndComp
 $Comp
-L VCC #PWR82
+L VCC #PWR075
 U 1 1 561D850D
 P 6900 3850
-F 0 "#PWR82" H 6900 3700 50  0001 C CNN
+F 0 "#PWR075" H 6900 3700 50  0001 C CNN
 F 1 "VCC" H 6900 4000 50  0000 C CNN
 F 2 "" H 6900 3850 60  0000 C CNN
@@
 	7200 1200 7550 1200
 $Comp
-L +15V #PWR90
+L +15V #PWR076
 U 1 1 561D8542
 P 8650 1700
-F 0 "#PWR90" H 8650 1550 50  0001 C CNN
+F 0 "#PWR076" H 8650 1550 50  0001 C CNN
 F 1 "+15V" H 8650 1840 50  0000 C CNN
 F 2 "" H 8650 1700 60  0000 C CNN
@@
 	10400 3800 10400 3750
 $Comp
-L GND-RESCUE-BatAger #PWR96
+L GND-RESCUE-BatAger #PWR077
 U 1 1 561D854D
 P 10400 4350
-F 0 "#PWR96" H 10400 4100 50  0001 C CNN
+F 0 "#PWR077" H 10400 4100 50  0001 C CNN
 F 1 "GND" H 10400 4200 50  0000 C CNN
 F 2 "" H 10400 4350 60  0000 C CNN
@@
 	8650 4250 8450 4250
 $Comp
-L VCC #PWR93
+L VCC #PWR078
 U 1 1 561D8558
 P 9500 3050
-F 0 "#PWR93" H 9500 2900 50  0001 C CNN
+F 0 "#PWR078" H 9500 2900 50  0001 C CNN
 F 1 "VCC" H 9500 3200 50  0000 C CNN
 F 2 "" H 9500 3050 60  0000 C CNN
@@
 +15V
 $Comp
-L +15V #PWR61
+L +15V #PWR079
 U 1 1 561DB3B7
 P 1400 5500
-F 0 "#PWR61" H 1400 5350 50  0001 C CNN
+F 0 "#PWR079" H 1400 5350 50  0001 C CNN
 F 1 "+15V" H 1400 5640 50  0000 C CNN
 F 2 "" H 1400 5500 60  0000 C CNN
@@
 VCC
 $Comp
-L GND-RESCUE-BatAger #PWR65
+L GND-RESCUE-BatAger #PWR080
 U 1 1 561DB84A
 P 1800 5900
-F 0 "#PWR65" H 1800 5650 50  0001 C CNN
+F 0 "#PWR080" H 1800 5650 50  0001 C CNN
 F 1 "GND" H 1800 5750 50  0000 C CNN
 F 2 "" H 1800 5900 60  0000 C CNN
@@
 $EndComp
 $Comp
-L VCC #PWR60
+L VCC #PWR081
 U 1 1 561DB968
 P 1300 6250
-F 0 "#PWR60" H 1300 6100 50  0001 C CNN
+F 0 "#PWR081" H 1300 6100 50  0001 C CNN
 F 1 "VCC" H 1300 6400 50  0000 C CNN
 F 2 "" H 1300 6250 60  0000 C CNN
@@
 	3200 5900 2800 5900
 $Comp
-L GND-RESCUE-BatAger #PWR72
+L GND-RESCUE-BatAger #PWR082
 U 1 1 561E128A
 P 3050 6150
-F 0 "#PWR72" H 3050 5900 50  0001 C CNN
+F 0 "#PWR082" H 3050 5900 50  0001 C CNN
 F 1 "GND" H 3050 6000 50  0000 C CNN
 F 2 "" H 3050 6150 60  0000 C CNN
@@
 	3200 6750 2800 6750
 $Comp
-L GND-RESCUE-BatAger #PWR73
+L GND-RESCUE-BatAger #PWR083
 U 1 1 561E13EC
 P 3050 7000
-F 0 "#PWR73" H 3050 6750 50  0001 C CNN
+F 0 "#PWR083" H 3050 6750 50  0001 C CNN
 F 1 "GND" H 3050 6850 50  0000 C CNN
 F 2 "" H 3050 7000 60  0000 C CNN
@@
 $EndComp
 $Comp
-L GND-RESCUE-BatAger #PWR67
+L GND-RESCUE-BatAger #PWR084
 U 1 1 561E41E4
 P 2100 4550
-F 0 "#PWR67" H 2100 4300 50  0001 C CNN
+F 0 "#PWR084" H 2100 4300 50  0001 C CNN
 F 1 "GND" H 2100 4400 50  0000 C CNN
 F 2 "" H 2100 4550 60  0000 C CNN
@@
 $EndComp
 $Comp
-L GND-RESCUE-BatAger #PWR66
+L GND-RESCUE-BatAger #PWR085
 U 1 1 561E448A
 P 2100 3050
-F 0 "#PWR66" H 2100 2800 50  0001 C CNN
+F 0 "#PWR085" H 2100 2800 50  0001 C CNN
 F 1 "GND" H 2100 2900 50  0000 C CNN
 F 2 "" H 2100 3050 60  0000 C CNN
@@
 $EndComp
 $Comp
-L GND-RESCUE-BatAger #PWR84
+L GND-RESCUE-BatAger #PWR086
 U 1 1 561E49F5
 P 7400 3050
-F 0 "#PWR84" H 7400 2800 50  0001 C CNN
+F 0 "#PWR086" H 7400 2800 50  0001 C CNN
 F 1 "GND" H 7400 2900 50  0000 C CNN
 F 2 "" H 7400 3050 60  0000 C CNN
@@
 $EndComp
 $Comp
-L GND-RESCUE-BatAger #PWR85
+L GND-RESCUE-BatAger #PWR087
 U 1 1 561E4C08
 P 7400 4700
-F 0 "#PWR85" H 7400 4450 50  0001 C CNN
+F 0 "#PWR087" H 7400 4450 50  0001 C CNN
 F 1 "GND" H 7400 4550 50  0000 C CNN
 F 2 "" H 7400 4700 60  0000 C CNN
@@
 $EndComp
 $Comp
-L GND-RESCUE-BatAger #PWR76
+L GND-RESCUE-BatAger #PWR088
 U 1 1 562667C6
 P 3950 2700
-F 0 "#PWR76" H 3950 2450 50  0001 C CNN
+F 0 "#PWR088" H 3950 2450 50  0001 C CNN
 F 1 "GND" H 3950 2550 50  0000 C CNN
 F 2 "" H 3950 2700 60  0000 C CNN
@@
 F 0 "C26" H 9210 2620 50  0000 L CNN
 F 1 "0.1uF" H 9210 2470 50  0000 L CNN
-F 2 "Capacitors_SMD:C_0805_HandSoldering" H 9200 2550 60  0001 C CNN
+F 2 "Capacitors_ThroughHole:C_Disc_D3_P2.5" H 9200 2550 60  0001 C CNN
 F 3 "" H 9200 2550 60  0000 C CNN
 	1    9200 2550
@@
 Connection ~ 9200 2400
 $Comp
-L GND-RESCUE-BatAger #PWR92
+L GND-RESCUE-BatAger #PWR089
 U 1 1 56266F2D
 P 9200 2750
-F 0 "#PWR92" H 9200 2500 50  0001 C CNN
+F 0 "#PWR089" H 9200 2500 50  0001 C CNN
 F 1 "GND" H 9200 2600 50  0000 C CNN
 F 2 "" H 9200 2750 60  0000 C CNN

Commit message: Minor package changes.
Parts:
- C25, C26: value 0.1uF -> 1uF
- P10, P11: footprint Pin_Headers:Pin_Header_Straight_1x02 -> Custom Footprints:PINHEAD1-2_200mil
- R47, R62: value 200 -> 15k
Changed lines of the file:
@@
 P 3650 2400
 F 0 "R47" V 3730 2400 50  0000 C CNN
-F 1 "200" V 3650 2400 50  0000 C CNN
+F 1 "15k" V 3650 2400 50  0000 C CNN
 F 2 "Resistors_SMD:R_0805_HandSoldering" V 3580 2400 30  0001 C CNN
 F 3 "" H 3650 2400 30  0000 C CNN
@@
 P 8900 2400
 F 0 "R62" V 8980 2400 50  0000 C CNN
-F 1 "200" V 8900 2400 50  0000 C CNN
+F 1 "15k" V 8900 2400 50  0000 C CNN
 F 2 "Custom Footprints:Resistor_Horizontal_RM10mm" V 8830 2400 30  0001 C CNN
 F 3 "" H 8900 2400 30  0000 C CNN
@@
 F 0 "P10" H 3400 6100 50  0000 C CNN
 F 1 "CONN_01X02" V 3500 5950 50  0000 C CNN
-F 2 "Pin_Headers:Pin_Header_Straight_1x02" H 3400 5950 60  0001 C CNN
+F 2 "Custom Footprints:PINHEAD1-2_200mil" H 3400 5950 60  0001 C CNN
 F 3 "" H 3400 5950 60  0000 C CNN
 	1    3400 5950
@@
 F 0 "P11" H 3400 6950 50  0000 C CNN
 F 1 "CONN_01X02" V 3500 6800 50  0000 C CNN
-F 2 "Pin_Headers:Pin_Header_Straight_1x02" H 3400 6800 60  0001 C CNN
+F 2 "Custom Footprints:PINHEAD1-2_200mil" H 3400 6800 60  0001 C CNN
 F 3 "" H 3400 6800 60  0000 C CNN
 	1    3400 6800
@@
 P 3950 2550
 F 0 "C25" H 3960 2620 50  0000 L CNN
-F 1 "0.1uF" H 3960 2470 50  0000 L CNN
+F 1 "1uF" H 3960 2470 50  0000 L CNN
 F 2 "Capacitors_SMD:C_0805_HandSoldering" H 3950 2550 60  0001 C CNN
 F 3 "" H 3950 2550 60  0000 C CNN
@@
 P 9200 2550
 F 0 "C26" H 9210 2620 50  0000 L CNN
-F 1 "0.1uF" H 9210 2470 50  0000 L CNN
+F 1 "1uF" H 9210 2470 50  0000 L CNN
 F 2 "Capacitors_ThroughHole:C_Disc_D3_P2.5" H 9200 2550 60  0001 C CNN
 F 3 "" H 9200 2550 60  0000 C CNN
